Commit message: Add files via upload

File: danphi_v2_description/urdf/danphi_v2.xacro (robot description, xacro)
@@ -8,5 +8,5 @@
     <parent link="base_footprint"/>
     <child link="base_link" />
-    <origin xyz="0 0 0.010" rpy="0 0 0"/>
+    <origin xyz="-2 1 0.010" rpy="0 0 0"/>
   </joint>
   <link name="base_link">
@@ -139,5 +139,5 @@
       <parent link="base_link"/>
       <child link="velodyne_base_link"/>
-	  <origin xyz="0 0 0.05867" rpy="0 0 0"/>
+	  <origin xyz="-0.0625 0 0.09375" rpy="0 0 0"/>
     </joint>
     <link name="velodyne_base_link">
@@ -188,5 +188,5 @@
             <scan>
               <horizontal>
-                <samples>2187</samples>
+                <samples>750<!--2187--></samples>
                 <resolution>1</resolution>
                 <min_angle>-${M_PI}</min_angle>
